Commit message: update urdf and rviz config file

File: urdf/robot_urdf.xacro (robot description, xacro)
@@ -190,4 +190,13 @@
     </gazebo> -->
     <!--  ########################### -->
+    <!--  IMU LINK -->
+    <joint name="imu_joint" type="fixed">
+        <parent link="chassis"/>
+        <child link="imu"/>
+        <origin xyz="0 0 ${chassis_height}"/>
+    </joint>
+    <link name="imu">
+    </link>
+    <!--  ########################### -->
     <!-- ############# add ros2_control => INSERT SMC_L298N_ROS_PLUGIN ############### -->
     <ros2_control name="smc_differential_drive_control" type="system">
@@ -197,5 +206,5 @@
         <param name="motorB_wheel_name">right_wheel_joint</param>
         <param name="port">/dev/ttyUSB0</param>
-        <!-- <param name="port">/dev/serial/by-path/platform-fd500000.pcie-pci-0000:01:00.0-usb-0:1.1.2:1.0-port0</param> -->
+        <!-- <param name="port">/dev/serial/by-path/pci-0000:00:14.0-usb-0:1.4:1.0-port0</param> -->
       </hardware>
       <joint name="left_wheel_joint">
